File: HW/Board/Board.sch (KiCad schematic (older format))
At the start: 1 part, among them J1 Screw_Terminal_01x02

Commit message: changed board around some, cleaned up libs
Connections:
- wire segments 7 -> 8
- no-connect marks 5 -> 6
Changed lines of the file:
@@
 EESchema Schematic File Version 4
-LIBS:Board-cache
-EELAYER 26 0
+EELAYER 30 0
 EELAYER END
 $Descr A4 11693 8268
@@
 F7 "CLK" I R 7900 1700 50
 F8 "DAC_CS" I R 7900 1350 50
+F9 "RELAIS" I L 6850 1700 50
 $EndSheet
 Wire Wire Line
@@
 	1    0    0    -1
 $EndComp
+NoConn ~ 6750 1700
+Wire Wire Line
+	6750 1700 6850 1700
 $EndSCHEMATC
