File: HW/Board/PowerChannel.sch (KiCad schematic (older format))
At the start: 33 parts, among them J2 Screw_Terminal_01x02, J4 Screw_Terminal_01x02, J5 Screw_Terminal_01x02, J6 Screw_Terminal_01x03, K1 FINDER-40.31, Q1 BC327, Q2 Q_NPN_BCE, U1 LM324, U2 INA219AIDCNR, U3 MCP4922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

Commit message: changed board around some, cleaned up libs
Parts:
- removed J4: Screw_Terminal_01x02, Connector_PinHeader_2.54mm:PinHeader_1x02_P2.54mm_Vertical, symbol Connector:Screw_Terminal_01x02
- removed J5: Screw_Terminal_01x02, Connector_PinHeader_2.54mm:PinHeader_1x03_P2.54mm_Vertical, symbol Connector:Screw_Terminal_01x03
- removed U4: LT1029, Package_TO_SOT_THT:TO-92, symbol Board-rescue:LT1029-Board
- removed U7: LM334Z_NOPB, digikey-footprints:TO-92-3, symbol Board-rescue:LM334Z_NOPB-dk_PMIC-Current-Regulation-Management
- added J3: Screw_Terminal_01x02, Connector_PinHeader_2.54mm:PinHeader_1x02_P2.54mm_Vertical, symbol Connector:Screw_Terminal_01x02
- added M1: LM2596-Buck, symbol Board:LM2596-Buck
- added Q3: BC327, Package_TO_SOT_THT:TO-92_Inline, symbol Transistor_BJT:BC327
- added U4: LM334Z, Package_TO_SOT_THT:TO-92_Inline, symbol Reference_Current:LM334Z
- added U7: LT1029, symbol Board:LT1029
Connections:
- net labels added: RELAIS
- net labels removed: +VDC, GNDA
- wire segments 126 -> 137
- no-connect marks 11 -> 9
Other:
- moved on the sheet: Q1
